Commit message: Update right/left hand urdf models

File: ros2_source/src/allegro_hand_description/urdf/allegro_hand_description_left.urdf (robot description, URDF)
Before this commit: robot allegro_hand_left, 21 links, 20 joints
Links:
- removed link link_0
- removed link link_1
- removed link link_10
- removed link link_11
- removed link link_11_tip
- removed link link_12
- removed link link_13
- removed link link_14
- removed link link_15
- removed link link_15_tip
- removed link link_2
- removed link link_3
- removed link link_3_tip
- removed link link_4
- removed link link_5
- removed link link_6
- removed link link_7
- removed link link_7_tip
- removed link link_8
- removed link link_9
- removed link palm_link
- added link base_link, mass 4.1685782e-01; collision mesh filename=package://allegro_hand_description/meshes/40_10_link_g_l.stl scale=0.001 0.001 0.001; visual mesh filename=package://allegro_hand_description/meshes/40_10_link_g_l.stl scale=0.001 0.001 0.001
- added link if1, mass 1.1350110e-02; collision mesh filename=package://allegro_hand_description/meshes/40_10_link_f1.stl scale=0.001 0.001 0.001; visual mesh filename=package://allegro_hand_description/meshes/40_10_link_f1.stl scale=0.001 0.001 0.001
- added link if2, mass 7.1189096e-02; collision mesh filename=package://allegro_hand_description/meshes/40_10_link_f2.stl scale=0.001 0.001 0.001; visual mesh filename=package://allegro_hand_description/meshes/40_10_link_f2.stl scale=0.001 0.001 0.001
- added link if3, mass 3.7588606e-02; collision mesh filename=package://allegro_hand_description/meshes/40_10_link_f3.stl scale=0.001 0.001 0.001; visual mesh filename=package://allegro_hand_description/meshes/40_10_link_f3.stl scale=0.001 0.001 0.001
- added link if4, mass 9.4301124e-03; collision mesh filename=package://allegro_hand_description/meshes/40_10_link_f4.stl scale=0.001 0.001 0.001; visual mesh filename=package://allegro_hand_description/meshes/40_10_link_f4.stl scale=0.001 0.001 0.001
- added link if5, mass 1.6654268e-02; collision mesh filename=package://allegro_hand_description/meshes/40_10_link_f5.stl scale=0.001 0.001 0.001; visual mesh filename=package://allegro_hand_description/meshes/40_10_link_f5.stl scale=0.001 0.001 0.001
- added link mf1, mass 1.1350110e-02; collision mesh filename=package://allegro_hand_description/meshes/40_10_link_f1.stl scale=0.001 0.001 0.001; visual mesh filename=package://allegro_hand_description/meshes/40_10_link_f1.stl scale=0.001 0.001 0.001
- added link mf2, mass 7.1189096e-02; collision mesh filename=package://allegro_hand_description/meshes/40_10_link_f2.stl scale=0.001 0.001 0.001; visual mesh filename=package://allegro_hand_description/meshes/40_10_link_f2.stl scale=0.001 0.001 0.001
- added link mf3, mass 3.7588606e-02; collision mesh filename=package://allegro_hand_description/meshes/40_10_link_f3.stl scale=0.001 0.001 0.001; visual mesh filename=package://allegro_hand_description/meshes/40_10_link_f3.stl scale=0.001 0.001 0.001
- added link mf4, mass 9.4301124e-03; collision mesh filename=package://allegro_hand_description/meshes/40_10_link_f4.stl scale=0.001 0.001 0.001; visual mesh filename=package://allegro_hand_description/meshes/40_10_link_f4.stl scale=0.001 0.001 0.001
- added link mf5, mass 1.6654268e-02; collision mesh filename=package://allegro_hand_description/meshes/40_10_link_f5.stl scale=0.001 0.001 0.001; visual mesh filename=package://allegro_hand_description/meshes/40_10_link_f5.stl scale=0.001 0.001 0.001
- added link pf1, mass 1.1350110e-02; collision mesh filename=package://allegro_hand_description/meshes/40_10_link_f1.stl scale=0.001 0.001 0.001; visual mesh filename=package://allegro_hand_description/meshes/40_10_link_f1.stl scale=0.001 0.001 0.001
- added link pf2, mass 7.1189096e-02; collision mesh filename=package://allegro_hand_description/meshes/40_10_link_f2.stl scale=0.001 0.001 0.001; visual mesh filename=package://allegro_hand_description/meshes/40_10_link_f2.stl scale=0.001 0.001 0.001
- added link pf3, mass 3.7588606e-02; collision mesh filename=package://allegro_hand_description/meshes/40_10_link_f3.stl scale=0.001 0.001 0.001; visual mesh filename=package://allegro_hand_description/meshes/40_10_link_f3.stl scale=0.001 0.001 0.001
- added link pf4, mass 9.4301124e-03; collision mesh filename=package://allegro_hand_description/meshes/40_10_link_f4.stl scale=0.001 0.001 0.001; visual mesh filename=package://allegro_hand_description/meshes/40_10_link_f4.stl scale=0.001 0.001 0.001
- added link pf5, mass 1.6654268e-02; collision mesh filename=package://allegro_hand_description/meshes/40_10_link_f5.stl scale=0.001 0.001 0.001; visual mesh filename=package://allegro_hand_description/meshes/40_10_link_f5.stl scale=0.001 0.001 0.001
- added link th1, mass 7.9809876e-02; collision mesh filename=package://allegro_hand_description/meshes/40_10_link_t1_l.s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 scale=0.001 0.001 0.001; visual mesh filename=package://allegro_hand_description/meshes/40_10_link_t1_l.s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 scale=0.001 0.001 0.001
- added link th2, mass 1.1350110e-02; collision mesh filename=package://allegro_hand_description/meshes/40_10_link_f1.stl scale=0.001 0.001 0.001; visual mesh filename=package://allegro_hand_description/meshes/40_10_link_f1.stl scale=0.001 0.001 0.001
- added link th3, mass 4.0206693e-02; collision mesh filename=package://allegro_hand_description/meshes/40_10_link_t3.stl scale=0.001 0.001 0.001; visual mesh filename=package://allegro_hand_description/meshes/40_10_link_t3.stl scale=0.001 0.001 0.001
- added link th4, mass  4.0750131e-02; collision mesh filename=package://allegro_hand_description/meshes/40_10_link_t4.stl scale=0.001 0.001 0.001; visual mesh filename=package://allegro_hand_description/meshes/40_10_link_t4.stl scale=0.001 0.001 0.001
- added link th5, mass 1.6654268e-02; collision mesh filename=package://allegro_hand_description/meshes/40_10_link_f5.stl scale=0.001 0.001 0.001; visual mesh filename=package://allegro_hand_description/meshes/40_10_link_f5.stl scale=0.001 0.001 0.001
Joints:
- removed joint joint_0
- removed joint joint_1
- removed joint joint_10
- removed joint joint_11
- removed joint joint_11_tip
- removed joint joint_12
- removed joint joint_13
- removed joint joint_14
- removed joint joint_15
- removed joint joint_15_tip
- removed joint joint_2
- removed joint joint_3
- removed joint joint_3_tip
- removed joint joint_4
- removed joint joint_5
- removed joint joint_6
- removed joint joint_7
- removed joint joint_7_tip
- removed joint joint_8
- removed joint joint_9
- added joint jif5: type fixed, parent pf4, child pf5, origin xyz=0.0157 0 0
- added joint jmf5: type fixed, parent mf4, child mf5, origin xyz=0.0157 0 0
- added joint joint_0.0: type revolute, parent base_link, child pf1, origin xyz=0 -0.045098 0.014293  rpy=0.0872665 0 0, axis 0 0 1, limit lower=-0.57 upper=0.57 effort=10 velocity=3
- added joint joint_1.0: type revolute, parent pf1, child pf2, origin xyz=0 0 0  rpy=0 0 0, axis 0 1 0, limit lower=-0.296 upper=1.71 effort=10 velocity=3
- added joint joint_10.0: type revolute, parent if2, child if3, origin xyz=0 0 0.054 rpy=0 -1.5708 0, axis 0 1 0, limit lower=-0.274 upper=1.809 effort=10 velocity=3
- added joint joint_11.0: type revolute, parent if3, child if4, origin xyz=0.0384 0 0, axis 0 1 0, limit lower=-0.327 upper=1.718 effort=10 velocity=3
- added joint joint_12.0: type revolute, parent base_link, child th1, origin xyz=-0.0182 -0.016958 -0.0723  rpy=0.0872665 0 0, axis 0 0 1, limit lower=0.36357 upper=1.4968 effort=10 velocity=3
- added joint joint_13.0: type revolute, parent th1, child th2, origin xyz=0.005 -0.055189 0  rpy=0 0 3.141593, axis 0 -1 0, limit lower=-0.20504289 upper=1.13 effort=10 velocity=3
- added joint joint_14.0: type revolute, parent th2, child th3, origin xyz=0 0 0  rpy=0 0 0, axis 1 0 0, limit lower=-0.2897 upper=1.633 effort=10 velocity=3
- added joint joint_15.0: type revolute, parent th3, child th4, origin xyz=0 0.051204 0  rpy=0 0 0, axis 1 0 0, limit lower=-0.2622 upper=1.81991 effort=10 velocity=3
- added joint joint_2.0: type revolute, parent pf2, child pf3, origin xyz=0 0 0.054 rpy=0 -1.5708 0, axis 0 1 0, limit lower=-0.274 upper=1.809 effort=10 velocity=3
- added joint joint_3.0: type revolute, parent pf3, child pf4, origin xyz=0.0384 0 0, axis 0 1 0, limit lower=-0.327 upper=1.718 effort=10 velocity=3
- added joint joint_4.0: type revolute, parent base_link, child mf1, origin xyz=0 0 0.0166 , axis 0 0 1, limit lower=-0.57 upper=0.57 effort=10 velocity=3
- added joint joint_5.0: type revolute, parent mf1, child mf2, origin xyz=0 0 0, axis 0 1 0, limit lower=-0.296 upper= 1.71 effort=10 velocity=3
- added joint joint_6.0: type revolute, parent mf2, child mf3, origin xyz=0 0 0.054 rpy=0 -1.5708 0, axis 0 1 0, limit lower=-0.274 upper= 1.809 effort=10 velocity=3
- added joint joint_7.0: type revolute, parent mf3, child mf4, origin xyz=0.0384 0 0 rpy=0 0 0, axis 0 1 0, limit lower=-0.327 upper=1.718 effort=10 velocity=3
- added joint joint_8.0: type revolute, parent base_link, child if1, origin xyz=0 0.045098 0.014293  rpy=-0.0872665 0 0, axis 0 0 1, limit lower=-0.57 upper=0.57 effort=10 velocity=3
- added joint joint_9.0: type revolute, parent if1, child if2, origin xyz=0 0 0  rpy=0 0 0, axis 0 1 0, limit lower=-0.296 upper=1.71 effort=10 velocity=3
- added joint jpf5: type fixed, parent if4, child if5, origin xyz=0.0157 0 0
- added joint jth5: type fixed, parent th4, child th5, origin xyz=0 0.0313 0  rpy=0 -1.4835335 0

File: ros2_source/src/allegro_hand_description/urdf/allegro_hand_description_right.urdf (robot description, URDF)
Before this commit: robot allegro_hand_right, 21 links, 20 joints
Links:
- removed link link_0
- removed link link_1
- removed link link_10
- removed link link_11
- removed link link_11_tip
- removed link link_12
- removed link link_13
- removed link link_14
- removed link link_15
- removed link link_15_tip
- removed link link_2
- removed link link_3
- removed link link_3_tip
- removed link link_4
- removed link link_5
- removed link link_6
- removed link link_7
- removed link link_7_tip
- removed link link_8
- removed link link_9
- removed link palm_link
- added link base_link, mass 4.1685782e-01; collision mesh filename=package://allegro_hand_description/meshes/40_10_link_g_r.stl scale=0.001 0.001 0.001; visual mesh filename=package://allegro_hand_description/meshes/40_10_link_g_r.stl scale=0.001 0.001 0.001
- added link if1, mass 1.1350110e-02; collision mesh filename=package://allegro_hand_description/meshes/40_10_link_f1.stl scale=0.001 0.001 0.001; visual mesh filename=package://allegro_hand_description/meshes/40_10_link_f1.stl scale=0.001 0.001 0.001
- added link if2, mass 7.1189096e-02; collision mesh filename=package://allegro_hand_description/meshes/40_10_link_f2.stl scale=0.001 0.001 0.001; visual mesh filename=package://allegro_hand_description/meshes/40_10_link_f2.stl scale=0.001 0.001 0.001
- added link if3, mass 3.7588606e-02; collision mesh filename=package://allegro_hand_description/meshes/40_10_link_f3.stl scale=0.001 0.001 0.001; visual mesh filename=package://allegro_hand_description/meshes/40_10_link_f3.stl scale=0.001 0.001 0.001
- added link if4, mass 9.4301124e-03; collision mesh filename=package://allegro_hand_description/meshes/40_10_link_f4.stl scale=0.001 0.001 0.001; visual mesh filename=package://allegro_hand_description/meshes/40_10_link_f4.stl scale=0.001 0.001 0.001
- added link if5, mass 1.6654268e-02; collision mesh filename=package://allegro_hand_description/meshes/40_10_link_f5.stl scale=0.001 0.001 0.001; visual mesh filename=package://allegro_hand_description/meshes/40_10_link_f5.stl scale=0.001 0.001 0.001
- added link mf1, mass 1.1350110e-02; collision mesh filename=package://allegro_hand_description/meshes/40_10_link_f1.stl scale=0.001 0.001 0.001; visual mesh filename=package://allegro_hand_description/meshes/40_10_link_f1.stl scale=0.001 0.001 0.001
- added link mf2, mass 7.1189096e-02; collision mesh filename=package://allegro_hand_description/meshes/40_10_link_f2.stl scale=0.001 0.001 0.001; visual mesh filename=package://allegro_hand_description/meshes/40_10_link_f2.stl scale=0.001 0.001 0.001
- added link mf3, mass 3.7588606e-02; collision mesh filename=package://allegro_hand_description/meshes/40_10_link_f3.stl scale=0.001 0.001 0.001; visual mesh filename=package://allegro_hand_description/meshes/40_10_link_f3.stl scale=0.001 0.001 0.001
- added link mf4, mass 9.4301124e-03; collision mesh filename=package://allegro_hand_description/meshes/40_10_link_f4.stl scale=0.001 0.001 0.001; visual mesh filename=package://allegro_hand_description/meshes/40_10_link_f4.stl scale=0.001 0.001 0.001
- added link mf5, mass 1.6654268e-02; collision mesh filename=package://allegro_hand_description/meshes/40_10_link_f5.stl scale=0.001 0.001 0.001; visual mesh filename=package://allegro_hand_description/meshes/40_10_link_f5.stl scale=0.001 0.001 0.001
- added link pf1, mass 1.1350110e-02; collision mesh filename=package://allegro_hand_description/meshes/40_10_link_f1.stl scale=0.001 0.001 0.001; visual mesh filename=package://allegro_hand_description/meshes/40_10_link_f1.stl scale=0.001 0.001 0.001
- added link pf2, mass 7.1189096e-02; collision mesh filename=package://allegro_hand_description/meshes/40_10_link_f2.stl scale=0.001 0.001 0.001; visual mesh filename=package://allegro_hand_description/meshes/40_10_link_f2.stl scale=0.001 0.001 0.001
- added link pf3, mass 3.7588606e-02; collision mesh filename=package://allegro_hand_description/meshes/40_10_link_f3.stl scale=0.001 0.001 0.001; visual mesh filename=package://allegro_hand_description/meshes/40_10_link_f3.stl scale=0.001 0.001 0.001
- added link pf4, mass 9.4301124e-03; collision mesh filename=package://allegro_hand_description/meshes/40_10_link_f4.stl scale=0.001 0.001 0.001; visual mesh filename=package://allegro_hand_description/meshes/40_10_link_f4.stl scale=0.001 0.001 0.001
- added link pf5, mass 1.6654268e-02; collision mesh filename=package://allegro_hand_description/meshes/40_10_link_f5.stl scale=0.001 0.001 0.001; visual mesh filename=package://allegro_hand_description/meshes/40_10_link_f5.stl scale=0.001 0.001 0.001
- added link th1, mass 7.9809876e-02; collision mesh filename=package://allegro_hand_description/meshes/40_10_link_t1_r.s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 scale=0.001 0.001 0.001; visual mesh filename=package://allegro_hand_description/meshes/40_10_link_t1_r.s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 scale=0.001 0.001 0.001
- added link th2, mass 1.1350110e-02; collision mesh filename=package://allegro_hand_description/meshes/40_10_link_f1.stl scale=0.001 0.001 0.001; visual mesh filename=package://allegro_hand_description/meshes/40_10_link_f1.stl scale=0.001 0.001 0.001
- added link th3, mass 4.0206693e-02; collision mesh filename=package://allegro_hand_description/meshes/40_10_link_t3.stl scale=0.001 0.001 0.001; visual mesh filename=package://allegro_hand_description/meshes/40_10_link_t3.stl scale=0.001 0.001 0.001
- added link th4, mass  4.0750131e-02; collision mesh filename=package://allegro_hand_description/meshes/40_10_link_t4.stl scale=0.001 0.001 0.001; visual mesh filename=package://allegro_hand_description/meshes/40_10_link_t4.stl scale=0.001 0.001 0.001
- added link th5, mass 1.6654268e-02; collision mesh filename=package://allegro_hand_description/meshes/40_10_link_f5.stl scale=0.001 0.001 0.001; visual mesh filename=package://allegro_hand_description/meshes/40_10_link_f5.stl scale=0.001 0.001 0.001
Joints:
- removed joint joint_11_tip
- removed joint joint_15_tip
- removed joint joint_3_tip
- removed joint joint_7_tip
- added joint jif5: type fixed, parent if4, child if5, origin xyz=0.0157 0 0
- added joint jmf5: type fixed, parent mf4, child mf5, origin xyz=0.0157 0 0
- added joint jpf5: type fixed, parent pf4, child pf5, origin xyz=0.0157 0 0
- added joint jth5: type fixed, parent th4, child th5, origin xyz=0 0.0313 0  rpy=0 -1.4835335 0
- joint joint_0.0: child link_0 -> if1; limit lower=-0.47 upper=0.47 effort=15 velocity=7 -> lower=-0.57 upper=0.57 effort=10 velocity=3; origin xyz=0 0.0435 0 rpy=-0.08726646255 0 0 -> xyz=0 0.045098 0.014293  rpy=-0.0872665 0 0; parent palm_link -> base_link
- joint joint_1.0: child link_1 -> if2; limit lower=-0.196 upper=1.61 effort=15 velocity=7 -> lower=-0.296 upper=1.71 effort=10 velocity=3; origin xyz=0 0 0.0164 -> xyz=0 0 0  rpy=0 0 0; parent link_0 -> if1
- joint joint_10.0: child link_10 -> pf3; limit lower=-0.174 upper=1.709 effort=15 velocity=7 -> lower=-0.274 upper=1.809 effort=10 velocity=3; origin xyz=0 0 0.054 -> xyz=0 0 0.054 rpy=0 -1.5708 0; parent link_9 -> pf2
- joint joint_11.0: child link_11 -> pf4; limit lower=-0.227 upper=1.618 effort=15 velocity=7 -> lower=-0.327 upper=1.718 effort=10 velocity=3; origin xyz=0 0 0.0384 -> xyz=0.0384 0 0; parent link_10 -> pf3
- joint joint_12.0: axis -1 0 0 -> 0 0 -1; child link_12 -> th1; limit lower=0.263 upper=1.396 effort=15 velocity=7 -> lower=0.36357 upper=1.4968 effort=10 velocity=3; origin xyz=-0.0182 0.019333 -0.045987 rpy=0 -1.65806278845 -1.5707963259 -> xyz=-0.0182 0.016958 -0.0723  rpy=-0.0872665 0 0; parent palm_link -> base_link
- joint joint_13.0: axis 0 0 1 -> 0 1 0; child link_13 -> th2; limit lower=-0.105 upper=1.163 effort=15 velocity=7 -> lower=-0.20504289 upper=1.13 effort=10 velocity=3; origin xyz=-0.027 0.005 0.0399 -> xyz=0.005 0.055189 0  rpy=0 0 0; parent link_12 -> th1
- joint joint_14.0: axis 0 1 0 -> 1 0 0; child link_14 -> th3; limit lower=-0.189 upper=1.644 effort=15 velocity=7 -> lower=-0.2897 upper=1.633 effort=10 velocity=3; origin xyz=0 0 0.0177 -> xyz=0 0 0  rpy=0 0 0; parent link_13 -> th2
- joint joint_15.0: axis 0 1 0 -> 1 0 0; child link_15 -> th4; limit lower=-0.162 upper=1.719 effort=15 velocity=7 -> lower=-0.2622 upper=1.81991 effort=10 velocity=3; origin xyz=0 0 0.0514 -> xyz=0 0.051204 0  rpy=0 0 0; parent link_14 -> th3
- joint joint_2.0: child link_2 -> if3; limit lower=-0.174 upper=1.709 effort=15 velocity=7 -> lower=-0.274 upper=1.809 effort=10 velocity=3; origin xyz=0 0 0.054 -> xyz=0 0 0.054 rpy=0 -1.5708 0; parent link_1 -> if2
- joint joint_3.0: child link_3 -> if4; limit lower=-0.227 upper=1.618 effort=15 velocity=7 -> lower=-0.327 upper=1.718 effort=10 velocity=3; origin xyz=0 0 0.0384 -> xyz=0.0384 0 0; parent link_2 -> if3
- joint joint_4.0: child link_4 -> mf1; limit lower=-0.47 upper=0.47 effort=15 velocity=7 -> lower=-0.57 upper=0.57 effort=10 velocity=3; origin xyz=0 0 0 rpy=0.0 0 0 -> xyz=0 0 0.0166 ; parent palm_link -> base_link
- joint joint_5.0: child link_5 -> mf2; limit lower=-0.196 upper=1.61 effort=15 velocity=7 -> lower=-0.296 upper= 1.71 effort=10 velocity=3; origin xyz=0 0 0.0164 -> xyz=0 0 0; parent link_4 -> mf1
- joint joint_6.0: child link_6 -> mf3; limit lower=-0.174 upper=1.709 effort=15 velocity=7 -> lower=-0.274 upper= 1.809 effort=10 velocity=3; origin xyz=0 0 0.054 -> xyz=0 0 0.054 rpy=0 -1.5708 0; parent link_5 -> mf2
- joint joint_7.0: child link_7 -> mf4; limit lower=-0.227 upper=1.618 effort=15 velocity=7 -> lower=-0.327 upper=1.718 effort=10 velocity=3; origin xyz=0 0 0.0384 -> xyz=0.0384 0 0 rpy=0 0 0; parent link_6 -> mf3
- joint joint_8.0: child link_8 -> pf1; limit lower=-0.47 upper=0.47 effort=15 velocity=7 -> lower=-0.57 upper=0.57 effort=10 velocity=3; origin xyz=0 -0.0435 0 rpy=0.08726646255 0 0 -> xyz=0 -0.045098 0.014293  rpy=0.0872665 0 0; parent palm_link -> base_link
- joint joint_9.0: child link_9 -> pf2; limit lower=-0.196 upper=1.61 effort=15 velocity=7 -> lower=-0.296 upper=1.71 effort=10 velocity=3; origin xyz=0 0 0.0164 -> xyz=0 0 0  rpy=0 0 0; parent link_8 -> pf1
